Commit message: updated b1_description

File: legged_examples/b1/b1_description/urdf/common/leg.xacro (robot description, xacro)
@@ -16,5 +16,5 @@
                 <origin rpy="0 0 0" xyz="${-leg_offset_x} ${leg_offset_y} 0"/>
             </xacro:if>
-            <parent link="trunk"/>
+            <parent link="base"/>
             <child link="${name}_hip"/>
             <axis xyz="1 0 0"/>
@@ -40,5 +40,5 @@
                 <origin rpy="0 0 0" xyz="${-hip_rotor_offset_x} ${hip_rotor_offset_y} 0"/>
             </xacro:if>
-            <parent link="trunk"/>
+            <parent link="base"/>
             <child link="${name}_hip_rotor"/>
         </joint>

File: legged_examples/b1/b1_description/urdf/robot.xacro (robot description, xacro)
@@ -6,21 +6,5 @@
     <xacro:include filename="$(find b1_description)/urdf/common/imu.xacro"/>
     <xacro:include filename="$(find b1_description)/urdf/b1/const.xacro"/>
-    <!-- Rotor related joint and link is only for demonstrate location. -->
-    <!-- Actually, the rotor will rotate and the joint is not fixed. Reduction ratio should be considered. -->
     <link name="base">
-        <visual>
-            <origin rpy="0 0 0" xyz="0 0 0"/>
-            <geometry>
-                <box size="0.001 0.001 0.001"/>
-            </geometry>
-        </visual>
-    </link>
-    <xacro:IMU connected_to="base" imu_name="unitree_imu" xyz="0. 0. 0." rpy="0. 0. 0."/>
-    <joint name="floating_base" type="fixed">
-        <origin rpy="0 0 0" xyz="0 0 0"/>
-        <parent link="base"/>
-        <child link="trunk"/>
-    </joint>
-    <link name="trunk">
         <visual>
             <origin rpy="0 0 0" xyz="0 0 0"/>

Commit message: b1 walking in legged_unitree_description

File: legged_examples/b1/b1_description/urdf/common/leg.xacro (robot description, xacro)
@@ -2,6 +2,7 @@
 <robot xmlns:xacro="http://www.ros.org/wiki/xacro">
     <xacro:include filename="$(find b1_description)/urdf/common/transmission.xacro"/>
-    <xacro:macro name="leg" params="name mirror mirror_dae front_hind front_hind_dae">
+    <xacro:macro name="leg" params="name mirror mirror_dae front_hind front_hind_dae *origin">
         <joint name="${name}_HAA" type="revolute">
+            <xacro:insert_block name="origin"/>
             <xacro:if value="${(mirror_dae == False) and (front_hind_dae == True)}">
                 <origin rpy="0 0 0" xyz="${leg_offset_x} ${-leg_offset_y} 0"/>

File: legged_examples/b1/b1_description/urdf/robot.xacro (robot description, xacro)
@@ -1,9 +1,10 @@
 <?xml version="1.0"?>
-<robot name="b1_description" xmlns:xacro="http://www.ros.org/wiki/xacro">
+<robot xmlns:xacro="http://www.ros.org/wiki/xacro" name="robot">
+    <xacro:arg name="robot_type" default="b1"/>
     <xacro:include filename="$(find b1_description)/urdf/common/materials.xacro"/>
     <xacro:include filename="$(find b1_description)/urdf/common/leg.xacro"/>
     <xacro:include filename="$(find b1_description)/urdf/common/gazebo.xacro"/>
     <xacro:include filename="$(find b1_description)/urdf/common/imu.xacro"/>
-    <xacro:include filename="$(find b1_description)/urdf/b1/const.xacro"/>
+    <xacro:include filename="$(find b1_description)/urdf/$(arg robot_type)/const.xacro"/>
     <link name="base">
         <visual>
