Commit message: updated b1_description

File: legged_examples/b1/b1_description/urdf/b1/const.xacro (robot description, xacro)
@@ -12,11 +12,12 @@
     <xacro:property name="thigh_shoulder_radius" value="0.044"/>
     <xacro:property name="thigh_shoulder_length" value="0.08"/>
+    <xacro:property name="thigh_shoulder_y_offset" value="-0.008"/>
     <xacro:property name="thigh_width" value="0.05"/>
     <xacro:property name="thigh_height" value="0.08"/>
+    <xacro:property name="thigh_x_offset" value="-0.015"/>
     <xacro:property name="calf_width" value="0.04"/>
     <xacro:property name="calf_height" value="0.05"/>
+    <xacro:property name="calf_x_offset" value="0.0"/>
     <xacro:property name="foot_radius" value="0.04"/>
-    <xacro:property name="stick_radius" value="0.01"/>
-    <xacro:property name="stick_length" value="0.2"/>
     <!-- kinematic value -->
     <xacro:property name="thigh_offset" value="0.12675"/>
@@ -29,19 +30,10 @@
     <xacro:property name="hip_offset" value="0.12675"/>
     <!-- offset of link and rotor locations (left front) -->
-    <xacro:property name="hip_offset_x" value="0.3455"/>
-    <xacro:property name="hip_offset_y" value="0.072"/>
-    <xacro:property name="hip_offset_z" value="0.0"/>
     <xacro:property name="hip_rotor_offset_x" value="0.1955"/>
     <xacro:property name="hip_rotor_offset_y" value="0.072"/>
     <xacro:property name="hip_rotor_offset_z" value="0.0"/>
-    <xacro:property name="thigh_offset_x" value="0"/>
-    <xacro:property name="thigh_offset_y" value="0.12675"/>
-    <xacro:property name="thigh_offset_z" value="0.0"/>
     <xacro:property name="thigh_rotor_offset_x" value="0.0"/>
     <xacro:property name="thigh_rotor_offset_y" value="0.00935"/>
     <xacro:property name="thigh_rotor_offset_z" value="0.0"/>
-    <xacro:property name="calf_offset_x" value="0.0"/>
-    <xacro:property name="calf_offset_y" value="0.0"/>
-    <xacro:property name="calf_offset_z" value="-0.35"/>
     <xacro:property name="calf_rotor_offset_x" value="0.0"/>
     <xacro:property name="calf_rotor_offset_y" value="-0.0519"/>
@@ -50,14 +42,14 @@
     <xacro:property name="damping" value="0"/>
     <xacro:property name="friction" value="0"/>
-    <xacro:property name="hip_position_max" value="0.75"/>
-    <xacro:property name="hip_position_min" value="-0.75"/>
+    <xacro:property name="hip_max" value="0.75"/>
+    <xacro:property name="hip_min" value="-0.75"/>
     <xacro:property name="hip_velocity_max" value="19.69"/>
     <xacro:property name="hip_torque_max" value="91.0035"/>
-    <xacro:property name="thigh_position_max" value="3.5"/>
-    <xacro:property name="thigh_position_min" value="-1.0"/>
+    <xacro:property name="thigh_max" value="3.5"/>
+    <xacro:property name="thigh_min" value="-1.0"/>
     <xacro:property name="thigh_velocity_max" value="23.32"/>
     <xacro:property name="thigh_torque_max" value="93.33"/>
-    <xacro:property name="calf_position_max" value="-0.6"/>
-    <xacro:property name="calf_position_min" value="-2.6"/>
+    <xacro:property name="calf_max" value="-0.6"/>
+    <xacro:property name="calf_min" value="-2.6"/>
     <xacro:property name="calf_velocity_max" value="15.55"/>
     <xacro:property name="calf_torque_max" value="140"/>
@@ -139,3 +131,14 @@
     <!-- foot -->
     <xacro:property name="foot_mass" value="0.05"/>
+    <!-- payload -->
+    <xacro:property name="payload_mass" value="3.0"/>
+    <xacro:property name="payload_x_offset" value="-0.15"/>
+    <xacro:property name="payload_y_offset" value="0.0"/>
+    <xacro:property name="payload_z_offset" value="0.25"/>
+    <xacro:property name="payload_ixx" value="0.009375"/>
+    <xacro:property name="payload_ixy" value="0.0"/>
+    <xacro:property name="payload_ixz" value="0.0"/>
+    <xacro:property name="payload_iyy" value="0.009375"/>
+    <xacro:property name="payload_iyz" value="0.0"/>
+    <xacro:property name="payload_izz" value="0.00375"/>
 </robot>

File: legged_examples/b1/b1_description/urdf/common/gazebo.xacro (robot description, xacro)
@@ -3,5 +3,5 @@
     <!-- ros_control plugin -->
     <gazebo>
-        <plugin name="gazebo_ros_control" filename="libgazebo_ros_control.so">
+        <plugin name="gazebo_ros_control" filename="liblegged_hw_sim.so">
             <robotNamespace>/</robotNamespace>
             <robotParam>b1_description</robotParam>

File: legged_examples/b1/b1_description/urdf/common/leg.xacro (robot description, xacro)
@@ -2,7 +2,6 @@
 <robot xmlns:xacro="http://www.ros.org/wiki/xacro">
     <xacro:include filename="$(find b1_description)/urdf/common/transmission.xacro"/>
-    <xacro:macro name="leg" params="name mirror mirror_dae front_hind front_hind_dae *origin">
-        <joint name="${name}_HAA" type="revolute">
-            <xacro:insert_block name="origin"/>
+    <xacro:macro name="leg" params="prefix mirror mirror_dae front_hind front_hind_dae *origin">
+        <joint name="${prefix}_HAA" type="revolute">
             <xacro:if value="${(mirror_dae == False) and (front_hind_dae == True)}">
                 <origin rpy="0 0 0" xyz="${leg_offset_x} ${-leg_offset_y} 0"/>
@@ -17,16 +16,19 @@
                 <origin rpy="0 0 0" xyz="${-leg_offset_x} ${leg_offset_y} 0"/>
             </xacro:if>
+            <xacro:insert_block name="origin"/>
             <parent link="base"/>
-            <child link="${name}_hip"/>
+            <child link="${prefix}_hip"/>
             <axis xyz="1 0 0"/>
             <dynamics damping="${damping}" friction="${friction}"/>
             <xacro:if value="${(mirror_dae == True)}">
-                <limit effort="${hip_torque_max}" velocity="${hip_velocity_max}" lower="${hip_position_min}" upper="${hip_position_max}"/>
+                <limit effort="${hip_torque_max}" velocity="${hip_velocity_max}" lower="${hip_min}"
+                       upper="${hip_max}"/>
             </xacro:if>
             <xacro:if value="${(mirror_dae == False)}">
-                <limit effort="${hip_torque_max}" velocity="${hip_velocity_max}" lower="${-hip_position_max}" upper="${-hip_position_min}"/>
-            </xacro:if>
-        </joint>
-        <joint name="${name}_hip_rotor_joint" type="fixed">
+                <limit effort="${hip_torque_max}" velocity="${hip_velocity_max}" lower="${-hip_max}"
+                       upper="${-hip_min}"/>
+            </xacro:if>
+        </joint>
+        <joint name="${prefix}_hip_rotor_joint" type="fixed">
             <xacro:if value="${(mirror_dae == False) and (front_hind_dae == True)}">
                 <origin rpy="0 0 0" xyz="${hip_rotor_offset_x} ${-hip_rotor_offset_y} 0"/>
@@ -42,7 +44,7 @@
             </xacro:if>
             <parent link="base"/>
-            <child link="${name}_hip_rotor"/>
-        </joint>
-        <link name="${name}_hip">
+            <child link="${prefix}_hip_rotor"/>
+        </joint>
+        <link name="${prefix}_hip">
             <visual>
                 <xacro:if value="${(mirror_dae == True) and (front_hind_dae == True)}">
@@ -50,19 +52,20 @@
                 </xacro:if>
                 <xacro:if value="${(mirror_dae == False) and (front_hind_dae == True)}">
-                    <origin rpy="${PI} 0 0" xyz="0 0 0"/>
+                    <origin rpy="${pi} 0 0" xyz="0 0 0"/>
                 </xacro:if>
                 <xacro:if value="${(mirror_dae == True) and (front_hind_dae == False)}">
-                    <origin rpy="0 ${PI} 0" xyz="0 0 0"/>
+                    <origin rpy="0 ${pi} 0" xyz="0 0 0"/>
                 </xacro:if>
                 <xacro:if value="${(mirror_dae == False) and (front_hind_dae == False)}">
-                    <origin rpy="${PI} ${PI} 0" xyz="0 0 0"/>
-                </xacro:if>
-                <geometry>
-                    <mesh filename="package://b1_description/meshes/hip.dae" scale="1 1 1"/>
-                </geometry>
-                <material name="orange"/>
-            </visual>
-            <collision>
-                <origin rpy="${PI/2.0} 0 0" xyz="0 ${hip_offset*mirror} 0"/>
+                    <origin rpy="${pi} ${pi} 0" xyz="0 0 0"/>
+                </xacro:if>
+                <geometry>
+                    <mesh filename="package://b1_description/meshes/$(arg robot_type)/hip.dae"
+                          scale="1 1 1"/>
+                </geometry>
+                <material name="orange"/>
+            </visual>
+            <collision>
+                <origin rpy="${pi/2.0} 0 0" xyz="0 0 0"/>
                 <geometry>
                     <cylinder length="${hip_length}" radius="${hip_radius}"/>
@@ -73,10 +76,10 @@
                 <mass value="${hip_mass}"/>
                 <inertia
-                    ixx="${hip_ixx}" ixy="${hip_ixy*mirror*front_hind}" ixz="${hip_ixz*front_hind}"
-                    iyy="${hip_iyy}" iyz="${hip_iyz*mirror}"
-                    izz="${hip_izz}"/>
-            </inertial>
-        </link>
-        <link name="${name}_hip_rotor">
+                        ixx="${hip_ixx}" ixy="${hip_ixy*mirror*front_hind}" ixz="${hip_ixz*front_hind}"
+                        iyy="${hip_iyy}" iyz="${hip_iyz*mirror}"
+                        izz="${hip_izz}"/>
+            </inertial>
+        </link>
+        <link name="${prefix}_hip_rotor">
             <visual>
                 <origin rpy="0 ${PI/2.0} 0" xyz="0 0 0"/>
@@ -86,10 +89,4 @@
                 <material name="green"/>
             </visual>
-            <!-- <collision>
-                <origin rpy="0 ${PI/2.0} 0" xyz="0 0 0"/>
-                <geometry>
-                    <cylinder length="0.02" radius="0.05"/>
-                </geometry>
-            </collision> -->
             <inertial>
                 <origin rpy="0 0 0" xyz="${hip_rotor_com_x} ${hip_rotor_com_y} ${hip_rotor_com_z}"/>
@@ -101,26 +98,29 @@
             </inertial>
         </link>
-        <joint name="${name}_HFE" type="revolute">
+        <joint name="${prefix}_HFE" type="revolute">
             <origin rpy="0 0 0" xyz="0 ${thigh_offset*mirror} 0"/>
-            <parent link="${name}_hip"/>
-            <child link="${name}_thigh"/>
+            <parent link="${prefix}_hip"/>
+            <child link="${prefix}_thigh"/>
             <axis xyz="0 1 0"/>
             <dynamics damping="${damping}" friction="${friction}"/>
-            <limit effort="${thigh_torque_max}" velocity="${thigh_velocity_max}" lower="${thigh_position_min}" upper="${thigh_position_max}"/>
-        </joint>
-        <joint name="${name}_thigh_rotor_joint" type="fixed">
+            <limit effort="${thigh_torque_max}" velocity="${thigh_velocity_max}" lower="${thigh_min}"
+                   upper="${thigh_max}"/>
+        </joint>
+        <joint name="${prefix}_thigh_rotor_joint" type="fixed">
             <origin rpy="0 0 0" xyz="${thigh_rotor_offset_x} ${thigh_rotor_offset_y*mirror} 0"/>
-            <parent link="${name}_hip"/>
-            <child link="${name}_thigh_rotor"/>
-        </joint>
-        <link name="${name}_thigh">
+            <parent link="${prefix}_hip"/>
+            <child link="${prefix}_thigh_rotor"/>
+        </joint>
+        <link name="${prefix}_thigh">
             <visual>
                 <origin rpy="0 0 0" xyz="0 0 0"/>
                 <geometry>
                     <xacro:if value="${mirror_dae == True}">
-                        <mesh filename="package://b1_description/meshes/thigh.dae" scale="1 1 1"/>
+                        <mesh filename="package://b1_description/meshes/$(arg robot_type)/thigh.dae"
+                              scale="1 1 1"/>
                     </xacro:if>
                     <xacro:if value="${mirror_dae == False}">
-                        <mesh filename="package://b1_description/meshes/thigh_mirror.dae" scale="1 1 1"/>
+                        <mesh filename="package://b1_description/meshes/$(arg robot_type)/thigh_mirror.dae"
+                              scale="1 1 1"/>
                     </xacro:if>
                 </geometry>
@@ -128,7 +128,13 @@
             </visual>
             <collision>
-                <origin rpy="0 ${PI/2.0} 0" xyz="0 0 ${-thigh_length/2.0}"/>
+                <origin rpy="0 ${pi/2.0+0.1} 0" xyz="${thigh_x_offset} 0 ${-thigh_length/2.0}"/>
                 <geometry>
                     <box size="${thigh_length} ${thigh_width} ${thigh_height}"/>
+                </geometry>
+            </collision>
+            <collision>
+                <origin rpy="${pi/2.0} 0 0" xyz="0 ${mirror*thigh_shoulder_y_offset} 0"/>
+                <geometry>
+                    <cylinder length="${thigh_shoulder_length}" radius="${thigh_shoulder_radius}"/>
                 </geometry>
             </collision>
@@ -137,10 +143,10 @@
                 <mass value="${thigh_mass}"/>
                 <inertia
-                    ixx="${thigh_ixx}" ixy="${thigh_ixy*mirror}" ixz="${thigh_ixz}"
-                    iyy="${thigh_iyy}" iyz="${thigh_iyz*mirror}"
-                    izz="${thigh_izz}"/>
-            </inertial>
-        </link>
-        <link name="${name}_thigh_rotor">
+                        ixx="${thigh_ixx}" ixy="${thigh_ixy*mirror}" ixz="${thigh_ixz}"
+                        iyy="${thigh_iyy}" iyz="${thigh_iyz*mirror}"
+                        izz="${thigh_izz}"/>
+            </inertial>
+        </link>
+        <link name="${prefix}_thigh_rotor">
             <visual>
                 <origin rpy="${PI/2.0} 0 0" xyz="0 0 0"/>
@@ -150,10 +156,4 @@
                 <material name="green"/>
             </visual>
-            <!-- <collision>
-                <origin rpy="${PI/2.0} 0 0" xyz="0 0 0"/>
-                <geometry>
-                    <cylinder length="0.02" radius="0.05"/>
-                </geometry>
-            </collision> -->
             <inertial>
                 <origin rpy="0 0 0" xyz="${thigh_rotor_com_x} ${thigh_rotor_com_y} ${thigh_rotor_com_z}"/>
@@ -165,27 +165,28 @@
             </inertial>
         </link>
-        <joint name="${name}_KFE" type="revolute">
+        <joint name="${prefix}_KFE" type="revolute">
             <origin rpy="0 0 0" xyz="0 0 ${-thigh_length}"/>
-            <parent link="${name}_thigh"/>
-            <child link="${name}_calf"/>
+            <parent link="${prefix}_thigh"/>
+            <child link="${prefix}_calf"/>
             <axis xyz="0 1 0"/>
             <dynamics damping="${damping}" friction="${friction}"/>
-            <limit effort="${calf_torque_max}" velocity="${calf_velocity_max}" lower="${calf_position_min}" upper="${calf_position_max}"/>
-        </joint>
-        <joint name="${name}_calf_rotor_joint" type="fixed">
+            <limit effort="${calf_torque_max}" velocity="${calf_velocity_max}" lower="${calf_min}" upper="${calf_max}"/>
+        </joint>
+        <joint name="${prefix}_calf_rotor_joint" type="fixed">
             <origin rpy="0 0 0" xyz="${calf_rotor_offset_x} ${calf_rotor_offset_y*mirror} 0"/>
-            <parent link="${name}_thigh"/>
-            <child link="${name}_calf_rotor"/>
-        </joint>
-        <link name="${name}_calf">
-            <visual>
-                <origin rpy="0 0 0" xyz="0 0 0"/>
-                <geometry>
-                    <mesh filename="package://b1_description/meshes/calf.dae" scale="1 1 1"/>
-                </geometry>
-                <material name="orange"/>
-            </visual>
-            <collision>
-                <origin rpy="0 ${PI/2.0} 0" xyz="0 0 ${-calf_length/2.0}"/>
+            <parent link="${prefix}_thigh"/>
+            <child link="${prefix}_calf_rotor"/>
+        </joint>
+        <link name="${prefix}_calf">
+            <visual>
+                <origin rpy="0 0 0" xyz="0 0 0"/>
+                <geometry>
+                    <mesh filename="package://b1_description/meshes/$(arg robot_type)/calf.dae"
+                          scale="1 1 1"/>
+                </geometry>
+                <material name="orange"/>
+            </visual>
+            <collision>
+                <origin rpy="0 ${pi/2.0} 0" xyz="${calf_x_offset} 0 ${-calf_length/2.0}"/>
                 <geometry>
                     <box size="${calf_length} ${calf_width} ${calf_height}"/>
@@ -196,10 +197,10 @@
                 <mass value="${calf_mass}"/>
                 <inertia
-                    ixx="${calf_ixx}" ixy="${calf_ixy}" ixz="${calf_ixz}"
-                    iyy="${calf_iyy}" iyz="${calf_iyz}"
-                    izz="${calf_izz}"/>
-            </inertial>
-        </link>
-        <link name="${name}_calf_rotor">
+                        ixx="${calf_ixx}" ixy="${calf_ixy}" ixz="${calf_ixz}"
+                        iyy="${calf_iyy}" iyz="${calf_iyz}"
+                        izz="${calf_izz}"/>
+            </inertial>
+        </link>
+        <link name="${prefix}_calf_rotor">
             <visual>
                 <origin rpy="${PI/2.0} 0 0" xyz="0 0 0"/>
@@ -209,10 +210,4 @@
                 <material name="green"/>
             </visual>
-            <!-- <collision>
-                <origin rpy="${PI/2.0} 0 0" xyz="0 0 0"/>
-                <geometry>
-                    <cylinder length="0.02" radius="0.05"/>
-                </geometry>
-            </collision> -->
             <inertial>
                 <origin rpy="0 0 0" xyz="${calf_rotor_com_x} ${calf_rotor_com_y} ${calf_rotor_com_z}"/>
@@ -224,10 +219,10 @@
             </inertial>
         </link>
-        <joint name="${name}_foot_fixed" type="fixed">
+        <joint name="${prefix}_foot_fixed" type="fixed">
             <origin rpy="0 0 0" xyz="0 0 ${-(calf_length)}"/>
-            <parent link="${name}_calf"/>
-            <child link="${name}_foot"/>
-        </joint>
-        <link name="${name}_FOOT">
+            <parent link="${prefix}_calf"/>
+            <child link="${prefix}_FOOT"/>
+        </joint>
+        <link name="${prefix}_FOOT">
             <visual>
                 <origin rpy="0 0 0" xyz="0 0 0"/>
@@ -235,5 +230,5 @@
                     <sphere radius="${foot_radius-0.01}"/>
                 </geometry>
-                <material name="green"/>
+                <material name="orange"/>
             </visual>
             <collision>
@@ -246,18 +241,18 @@
                 <mass value="${foot_mass}"/>
                 <inertia
-                    ixx="${(2*foot_mass)/5.0*(foot_radius*foot_radius)}" ixy="0.0" ixz="0.0"
-                    iyy="${(2*foot_mass)/5.0*(foot_radius*foot_radius)}" iyz="0.0"
-                    izz="${(2*foot_mass)/5.0*(foot_radius*foot_radius)}"/>
-            </inertial>
-        </link>
-        <gazebo reference="${name}_foot_fixed">
+                        ixx="${(2*foot_mass)/5.0*(foot_radius*foot_radius)}" ixy="0.0" ixz="0.0"
+                        iyy="${(2*foot_mass)/5.0*(foot_radius*foot_radius)}" iyz="0.0"
+                        izz="${(2*foot_mass)/5.0*(foot_radius*foot_radius)}"/>
+            </inertial>
+        </link>
+        <gazebo reference="${prefix}_foot_fixed">
             <disableFixedJointLumping>true</disableFixedJointLumping>
         </gazebo>
-        <gazebo reference="${name}_hip">
+        <gazebo reference="${prefix}_hip">
             <mu1>0.2</mu1>
             <mu2>0.2</mu2>
             <material>Gazebo/DarkGrey</material>
         </gazebo>
-        <gazebo reference="${name}_thigh">
+        <gazebo reference="${prefix}_thigh">
             <mu1>0.2</mu1>
             <mu2>0.2</mu2>
@@ -267,10 +262,10 @@
             <kd value="100.0"/>
         </gazebo>
-        <gazebo reference="${name}_calf">
+        <gazebo reference="${prefix}_calf">
             <mu1>0.6</mu1>
             <mu2>0.6</mu2>
             <self_collide>1</self_collide>
         </gazebo>
-        <gazebo reference="${name}_FOOT">
+        <gazebo reference="${prefix}_FOOT">
             <mu1>0.6</mu1>
             <mu2>0.6</mu2>
@@ -280,5 +275,5 @@
             <kd value="100.0"/>
         </gazebo>
-        <xacro:leg_transmission name="${name}"/>
+        <xacro:leg_transmission name="${prefix}"/>
     </xacro:macro>
 </robot>

File: legged_examples/b1/b1_description/urdf/common/transmission.xacro (robot description, xacro)
@@ -2,32 +2,32 @@
 <robot xmlns:xacro="http://www.ros.org/wiki/xacro">
     <xacro:macro name="leg_transmission" params="name">
-        <transmission name="${name}_HAA_tran">
+        <transmission name="${prefix}_HAA_tran">
             <type>transmission_interface/SimpleTransmission</type>
-            <joint name="${name}_HAA_joint">
-            <hardwareInterface>hardware_interface/EffortJointInterface</hardwareInterface>
+            <joint name="${prefix}_HAA">
+                <hardwareInterface>hardware_interface/EffortJointInterface</hardwareInterface>
             </joint>
-            <actuator name="${name}_HAA_motor">
-            <hardwareInterface>hardware_interface/EffortJointInterface</hardwareInterface>
-            <mechanicalReduction>1</mechanicalReduction>
+            <actuator name="${prefix}_HAA_motor">
+                <hardwareInterface>hardware_interface/EffortJointInterface</hardwareInterface>
+                <mechanicalReduction>1</mechanicalReduction>
             </actuator>
         </transmission>
-        <transmission name="${name}_HFE_tran">
+        <transmission name="${prefix}_HFE_tran">
             <type>transmission_interface/SimpleTransmission</type>
-            <joint name="${name}_HFE_joint">
-            <hardwareInterface>hardware_interface/EffortJointInterface</hardwareInterface>
+            <joint name="${prefix}_HFE">
+                <hardwareInterface>hardware_interface/EffortJointInterface</hardwareInterface>
             </joint>
-            <actuator name="${name}_HFE_motor">
-            <hardwareInterface>hardware_interface/EffortJointInterface</hardwareInterface>
-            <mechanicalReduction>1</mechanicalReduction>
+            <actuator name="${prefix}_HFE_motor">
+                <hardwareInterface>hardware_interface/EffortJointInterface</hardwareInterface>
+                <mechanicalReduction>1</mechanicalReduction>
             </actuator>
         </transmission>
-        <transmission name="${name}_KFE_tran">
+        <transmission name="${prefix}_KFE_tran">
             <type>transmission_interface/SimpleTransmission</type>
-            <joint name="${name}_KFE_joint">
-            <hardwareInterface>hardware_interface/EffortJointInterface</hardwareInterface>
+            <joint name="${prefix}_KFE">
+                <hardwareInterface>hardware_interface/EffortJointInterface</hardwareInterface>
             </joint>
-            <actuator name="${name}_KFE_motor">
-            <hardwareInterface>hardware_interface/EffortJointInterface</hardwareInterface>
-            <mechanicalReduction>1</mechanicalReduction>
+            <actuator name="${prefix}_KFE_motor">
+                <hardwareInterface>hardware_interface/EffortJointInterface</hardwareInterface>
+                <mechanicalReduction>1</mechanicalReduction>
             </actuator>
         </transmission>
